File: electonics/board/NaMi_Menu_v2.kicad_pcb (KiCad board)
At the start: 2 copper layers, 132 x 37.5 mm, 44 parts, among them J1 Conn_01x06, J10 Conn_01x02, J11 Conn_01x02, J12 Conn_01x02, J13 Conn_01x02, J2 Conn_01x03, J3 Conn_01x02, J4 Conn_01x02, J5 Conn_02x08_Odd_Even, J6 Conn_01x02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

Commit message: Modified PCB design
Parts:
- removed the H2 at (157.0, 55.0)
- removed the H3 at (157.0, 83.5)
- removed the J2 at (133.4, 79.0)
- added G***: LOGO, Symbol:NaMi-logo, B.Cu at (102.9, 83.0)
- added J5: Conn_01x02, Connector_PinHeader_2.54mm:PinHeader_1x02_P2.54mm_Vertical, B.Cu at (128.8, 55.2)
- C1, C2, C3, C4, C6, C7, C8, C9, U2: moved to B.Cu
- J3: value Conn_01x02 -> Conn_01x03; footprint Connector_PinHeader_2.54mm:PinHeader_1x02_P2.54mm_Vertical -> Connector_PinHeader_2.54mm:PinHeader_1x03_P2.54mm_Vertical
- L1: footprint Inductor_SMD:L_0805_2012Metric -> Inductor_SMD:L_Neosid_SMs42; moved to B.Cu
- R10, R11, R12, R7, R8, R9: value 100R -> 1k
- moved C5 51.0 mm to (120.2, 60.9)
- moved D1 44.7 mm to (172.5, 85.8), turned to -90 degrees
- moved J3 43.4 mm to (117.1, 82.8), turned to 90 degrees
- moved R7 43.0 mm to (89.5, 62.0), turned to 90 degrees
- moved C4 41.8 mm to (107.2, 70.5), turned to 0 degrees
- moved R6 41.6 mm to (107.1, 72.8), turned to 180 degrees
- moved R12 40.5 mm to (169.6, 85.8), turned to -90 degrees
- moved R8 38.9 mm to (94.1, 62.0), turned to 90 degrees
- moved L1 37.8 mm to (113.3, 62.2)
- moved R5 35.7 mm to (173.5, 82.0), turned to 90 degrees
- moved R9 35.0 mm to (98.6, 62.0), turned to 90 degrees
- moved J9 34.7 mm to (89.5, 55.2), turned to 180 degrees
- moved C6 32.9 mm to (117.7, 60.9), turned to 90 degrees
- moved C3 31.6 mm to (168.5, 82.0), turned to -90 degrees
- moved C2 31.5 mm to (178.5, 57.0), turned to -90 degrees
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- renumbered H4 to H2, H5 to H3, H6 to H4, J5 to J2
Connections:
- J3 pad 1: BTN1 -> GND
- J3 pad 2: VCC -> SWCLK
- J4 pad 1: BTN2 -> GND
- J4 pad 2: VCC -> BTN1
- J6 pad 1: BTN3 -> GND
- J6 pad 2: VCC -> BTN3
- J7 pad 1: BTN4 -> GND
- J7 pad 2: VCC -> BTN4
- J8 pad 1: BTN5 -> GND
- J8 pad 2: VCC -> BTN5
Routing:
- net SIG A OUT: track 9.49 -> 69.5 mm
- net INTERRUPT: track 45.9 -> 90.7 mm, vias 1 -> 6
- net MISO: track 51.0 -> 92.7 mm, vias 1 -> 6
- net SIG B OUT: track 15.8 -> 54.6 mm, vias 4 -> 2
- net SCK: track 57.5 -> 91.3 mm, vias 1 -> 5
- net CS: track 57.8 -> 88.4 mm, vias 2 -> 5
- net CS_OLED: track 20.2 -> 49.0 mm, vias 0 -> 1
- net DC_OLED: track 17.3 -> 45.5 mm, vias 0 -> 1
- net Net-(U2-GPIO15): track 7.94 -> 35.6 mm, vias 1 -> 2
- net S1: track 38.6 -> 65.8 mm, vias 5 -> 4
- net MOSI: track 57.9 -> 84.8 mm, vias 2 -> 4
- net RESET_OLED: track 17.3 -> 42.7 mm
- net Net-(VR1-A): track 32.3 -> 7.94 mm
- net Net-(VR1-B): track 30.4 -> 7.54 mm
- net BTN5: track 13.9 -> 35.5 mm
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- added copper zone on B.Cu, net GND
- removed copper zone on F.Cu, net GND
Other:
- board text added: "BTN"
- board text added: "GND"
- board text added: "Jakub Naumowicz"
- board text added: "KN NaMi"
- board text added: "LED"
- board text added: "NaMi-Menu v2.0"
- board text added: "Szymon Butkiewicz"

Commit message: PCB Correction + Gerber files
Parts:
- moved C1 40.5 mm to (191.7, 86.1)
- moved C2 40.5 mm to (206.7, 86.1)
- moved C3 40.5 mm to (196.7, 111.1)
- moved C4 40.5 mm to (135.3, 99.7), turned to 180 degrees
- moved C7 40.5 mm to (155.4, 104.8)
- moved C8 40.5 mm to (155.4, 101.8)
- moved D1 40.5 mm to (200.7, 114.9)
- moved H1 40.5 mm to (213.2, 84.1)
- moved H2 40.5 mm to (213.2, 112.6)
- moved H3 40.5 mm to (90.2, 84.1)
- moved H4 40.5 mm to (90.2, 112.6)
- moved J10 40.5 mm to (122.2, 84.4)
- moved J2 40.5 mm to (183.9, 107.2)
- moved J3 40.5 mm to (145.2, 112.0)
- moved J9 40.5 mm to (117.7, 84.4)
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Routing:
- net VCC: track 151.7 -> 159.5 mm, vias 13 -> 12
- net GND: track 20.0 -> 15.9 mm, vias 3 -> 2
- net SCK: track 91.3 -> 94.3 mm, vias 5 -> 3
- net MOSI: track 84.8 -> 86.6 mm, vias 4 -> 2
- net INTERRUPT: track 90.7 -> 92.3 mm, vias 6 -> 2
- net CS: track 88.4 -> 89.8 mm, vias 5 -> 3
- net MISO: track 92.7 -> 94.0 mm, vias 6 -> 2
- net Net-(U2-VREG_AVDD): track 8.30 -> 7.13 mm
- net CS_OLED: track 49.0 -> 49.9 mm
- net S1: track 65.8 -> 65.6 mm, vias 4 -> 2
Other:
- board text added: "BTN1"
- board text added: "BTN2"
- board text added: "BTN3"
- board text added: "BTN4"
- board text added: "BTN5"
- board text added: "CLK"
- board text added: "LED1"
- board text added: "LED2"
- board text added: "LED3"
- board text added: "LED4"
- board text added: "LED5"
- board text added: "SWD"
- board text removed: "BTN"
- board text removed: "LED"
